File: barometer.kicad_sch (KiCad schematic)
At the start: 0 parts

Commit message: update sensors
Other:
- company: (none) -> UCSC Rocket Team
- title: (none) -> Barometer
Changed lines of the file:
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@@
 	(generator_version "9.0")
 	(paper "A4")
+	(title_block
+		(title "Barometer")
+		(company "UCSC Rocket Team")
+	)
 )
