File: barometer.kicad_sch (KiCad schematic)
At the start: 2 parts, among them U5 MS5611

Commit message: Connected topsheet
Changed lines of the file:
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@@
 	)
 	(hierarchical_label "MISO"
-		(shape input)
+		(shape output)
 		(at 102.87 74.93 180)
 		(effects
@@
 		)
 	)
-	(hierarchical_label "3V3"
+	(hierarchical_label "+3V3"
 		(shape input)
 		(at 80.01 58.42 180)

Commit message: Footprint selection
Parts:
- C15: footprint (none) -> Capacitor_SMD:C_0603_1608Metric
- U5: footprint (none) -> Avionics_Feet:XDCR_MS561101BA03-50
Changed lines of the file:
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@@
 			)
 		)
-		(property "Footprint" ""
+		(property "Footprint" "Capacitor_SMD:C_0603_1608Metric"
 			(at 80.01 60.96 0)
 			(effects
@@
 			)
 		)
-		(property "Footprint" ""
+		(property "Footprint" "Avionics_Feet:XDCR_MS561101BA03-50"
 			(at 115.57 90.17 0)
 			(effects

Commit message: Radio footprint selection
Parts:
- renumbered C15 to C17, U5 to U6
Changed lines of the file:
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@@
 		(dnp no)
 		(fields_autoplaced yes)
-		(property "Reference" "C15"
+		(property "Reference" "C17"
 			(at 82.55 59.6962 0)
 			(effects
@@
 			(project ""
 				(path "/2c2eadf0-5503-4531-8753-1a232087fe8c/b9b0c40a-7771-4bc1-adbf-abe0201c34d0/9ad84ef5-c94d-4ded-9701-2036daea17e6"
-					(reference "C15")
+					(reference "C17")
 					(unit 1)
 				)
@@
 		(dnp no)
 		(fields_autoplaced yes)
-		(property "Reference" "#PWR064"
+		(property "Reference" "#PWR070"
 			(at 80.01 62.23 0)
 			(effects
@@
 			(project ""
 				(path "/2c2eadf0-5503-4531-8753-1a232087fe8c/b9b0c40a-7771-4bc1-adbf-abe0201c34d0/9ad84ef5-c94d-4ded-9701-2036daea17e6"
-					(reference "#PWR064")
+					(reference "#PWR070")
 					(unit 1)
 				)
@@
 		(dnp no)
 		(fields_autoplaced yes)
-		(property "Reference" "#PWR067"
+		(property "Reference" "#PWR073"
 			(at 120.65 86.36 0)
 			(effects
@@
 			(project "Blaze-NT"
 				(path "/2c2eadf0-5503-4531-8753-1a232087fe8c/b9b0c40a-7771-4bc1-adbf-abe0201c34d0/9ad84ef5-c94d-4ded-9701-2036daea17e6"
-					(reference "#PWR067")
+					(reference "#PWR073")
 					(unit 1)
 				)
@@
 		(dnp no)
 		(fields_autoplaced yes)
-		(property "Reference" "U5"
+		(property "Reference" "U6"
 			(at 111.76 59.69 0)
 			(effects
@@
 			(project ""
 				(path "/2c2eadf0-5503-4531-8753-1a232087fe8c/b9b0c40a-7771-4bc1-adbf-abe0201c34d0/9ad84ef5-c94d-4ded-9701-2036daea17e6"
-					(reference "U5")
+					(reference "U6")
 					(unit 1)
 				)
@@
 		(dnp no)
 		(fields_autoplaced yes)
-		(property "Reference" "#PWR065"
+		(property "Reference" "#PWR071"
 			(at 80.01 69.85 0)
 			(effects
@@
 			(project ""
 				(path "/2c2eadf0-5503-4531-8753-1a232087fe8c/b9b0c40a-7771-4bc1-adbf-abe0201c34d0/9ad84ef5-c94d-4ded-9701-2036daea17e6"
-					(reference "#PWR065")
+					(reference "#PWR071")
 					(unit 1)
 				)
@@
 		(dnp no)
 		(fields_autoplaced yes)
-		(property "Reference" "#PWR066"
+		(property "Reference" "#PWR072"
 			(at 102.87 71.12 0)
 			(effects
@@
 			(project "Blaze-NT"
 				(path "/2c2eadf0-5503-4531-8753-1a232087fe8c/b9b0c40a-7771-4bc1-adbf-abe0201c34d0/9ad84ef5-c94d-4ded-9701-2036daea17e6"
-					(reference "#PWR066")
-					(unit 1)
-				)
+					(reference "#PWR072")
+					(unit 1)
+				)

Commit message: Addeed part numbers
Parts:
- C17: LCSC (none) -> C14663
- U6: LCSC (none) -> C15639
Changed lines of the file:
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@@
+			)
+		)
+		(property "LCSC" "C14663"
+			(at 80.01 60.96 0)
+			(effects
+				(font
+					(size 1.27 1.27)
+				)
+				(hide yes)
 			)
 		)
@@
 			(effects
 				(font
+					(size 1.27 1.27)
+				)
+				(hide yes)
+			)
+		)
+		(property "LCSC" "C15639"
+			(at 111.76 73.66 0)
+			(effects
+				(font

Commit message: Added Digikey Components
Parts:
- U6: Digikey (none) -> MS561101BA03-50
Changed lines of the file:
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@@
+			)
+		)
+		(property "Digikey" ""
+			(at 80.01 60.96 0)
+			(effects
+				(font
+					(size 1.27 1.27)
+				)
+				(hide yes)
 			)
 		)
@@
 			(at 111.76 73.66 0)
 			(effects
+				(font
+					(size 1.27 1.27)
+				)
+				(hide yes)
+			)
+		)
+		(property "Digikey" "MS561101BA03-50"
+			(at 111.76 73.66 0)
+			(effects
