File: imu.kicad_sch (KiCad schematic)
At the start: 0 parts

Commit message: update sensors
Other:
- company: (none) -> UCSC Rocket Team
- title: (none) -> IMU
Changed lines of the file:
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@@
 	(generator_version "9.0")
 	(paper "A4")
+	(title_block
+		(title "IMU")
+		(company "UCSC Rocket Team")
+	)
 )

Commit message: save changes
Parts:
- added U4: LSM9DS1, symbol Avionics_Symbols:lsm9ds1
Connections:
- new net +3V3: U4.1 (VIN), U4.2 (3V3)
- new net CS_IMU_AG: U4.6 (CSAG)
- new net CS_IMU_MAG: U4.7 (CSM)
- new net GND: U4.3 (GND)
- new net MISO_AG: U4.8 (SDOAG)
- new net MISO_MAG: U4.9 (SDOM)
- new net MOSI: U4.5 (SDA/MOSI)
- new net SCK: U4.4 (SCL)
