File: accelerometer.kicad_sch (KiCad schematic)
At the start: 0 parts

Commit message: update sensors
Other:
- company: (none) -> UCSC Rocket Team
- title: (none) -> Accelerometer
Changed lines of the file:
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@@
 	(generator_version "9.0")
 	(paper "A4")
+	(title_block
+		(title "Accelerometer")
+		(company "UCSC Rocket Team")
+	)
 )

Commit message: random
Parts:
- added U4: kx13x, symbol Avionics_Symbols:kx13x
Connections:
- new net 3V3: U4.2 (3V3)
- new net CS_ACCEL: U4.6 (nCS)
- new net GND: U4.1 (GND)
- new net MISO: U4.5 (ADR/SDO)
- new net MOSI: U4.3 (SDA/SDI)
- new net SCK: U4.4 (SCL/SCLK)
- no-connect marks 0 -> 3
Changed lines of the file:
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@@
 		(company "UCSC Rocket Team")
 	)
+	(no_connect
+		(at 160.02 92.71)
+	)
+	(no_connect
+		(at 160.02 90.17)
+	)
+	(no_connect
+		(at 160.02 95.25)
+	)
+	(hierarchical_label "GND"
+		(shape input)
+		(at 160.02 102.87 0)
+		(effects
+			(font
+				(size 1.27 1.27)
+			)
+			(justify left)
+		)
+	)
+	(hierarchical_label "SCK"
+		(shape input)
+		(at 137.16 100.33 180)
+		(effects
+			(font
+				(size 1.27 1.27)
+			)
+			(justify right)
+		)
+	)
+	(hierarchical_label "3V3"
+		(shape input)
+		(at 137.16 90.17 180)
+		(effects
+			(font
+				(size 1.27 1.27)
+			)
+			(justify right)
+		)
+	)
+	(hierarchical_label "CS_ACCEL"
+		(shape input)
+		(at 137.16 102.87 180)
+		(effects
+			(font
+				(size 1.27 1.27)
+			)
+			(justify right)
+		)
+	)
+	(hierarchical_label "MOSI"
+		(shape input)
+		(at 137.16 95.25 180)
+		(effects
+			(font
+				(size 1.27 1.27)
+			)
+			(justify right)
+		)
+	)
+	(hierarchical_label "MISO"
+		(shape input)
+		(at 137.16 97.79 180)
+		(effects
+			(font
+				(size 1.27 1.27)
+			)
+			(justify right)
+		)
+	)
+	(symbol
+		(lib_id "Avionics_Symbols:kx13x")
+		(at 148.59 96.52 0)
+		(unit 1)
+		(exclude_from_sim no)
+		(in_bom yes)
+		(on_board yes)
+		(dnp no)
+		(fields_autoplaced yes)
+		(property "Reference" "U4"
+			(at 148.59 82.55 0)
+			(effects
+				(font
+					(size 1.27 1.27)
+				)
+			)
+		)
+		(property "Value" "kx13x"
+			(at 148.59 85.09 0)
+			(effects
+				(font
+					(size 1.27 1.27)
+				)
+			)
+		)
+		(property "Footprint" ""
+			(at 127 83.82 0)
+			(effects
+				(font
+					(size 1.27 1.27)
+				)
+				(hide yes)
+			)
+		)
+		(property "Datasheet" ""
+			(at 127 83.82 0)
+			(effects
+				(font
+					(size 1.27 1.27)
+				)
+				(hide yes)
+			)
+		)
+		(property "Description" ""
+			(at 127 83.82 0)
+			(effects
+				(font
+					(size 1.27 1.27)
+				)
+				(hide yes)
+			)
+		)
+		(pin "6"
+		)
+		(pin "7"
+		)
+		(pin "2"
+		)
+		(pin "5"
+		)
+		(pin "8"
+		)
+		(pin "1"
+		)
+		(pin "9"
+		)
+		(pin "3"
+		)
+		(pin "4"
+		)
+		(instances
+			(project ""
+				(path "/2c2eadf0-5503-4531-8753-1a232087fe8c/b9b0c40a-7771-4bc1-adbf-abe0201c34d0/9a6553ac-59f7-4d16-afa0-9743f2c46ffa"
+					(reference "U4")
+					(unit 1)
+				)
+			)
+		)
+	)
 )
