File: Blaze-NT.kicad_pcb (KiCad board)
At the start: 2 copper layers, 44.4 x 44.7 mm, 78 parts, among them J1 Micro_SD_Card, J2 TC2030-NL, J3 USB_C_Receptacle, J4 ARM, J5 BATTERY, J6 Stemma, SW1 SW_SPST, SW2 SW_SPST, U1 W25Q128JVS, U2 STM32F411CEUx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

Commit message: Silk updates
Other:
- board text added: "BLAZE NT B"
- board text removed: "BLAZE NT"
Changed lines of the file:
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@@
 			(at 0.025 -1.875 0)
 			(layer "F.SilkS")
+			(hide yes)
 			(effects
 				(font
@@
 		)
 	)
-	(gr_text "BLAZE NT"
-		(at 152.781 119.888 0)
+	(gr_text "BLAZE NT B"
+		(at 152.5016 119.8372 0)
 		(layer "F.SilkS")
 		(effects
